Commit message: switch roundr_description build_type to ament_cmake; complete urdf

File: roundr_description/urdf/roundr.urdf (robot description, URDF)
Before this commit: robot roundr, 6 links, 5 joints
Links:
- removed link chassis
- added link base_footprint
- added link base_inertial
- added link base_link; collision cylinder length=${base_width} radius=${base_radius}; visual cylinder length=${base_width} radius=${base_radius}
- link caster: mass 0.004 -> None; geometry collision sphere radius=${caster_radius}; visual sphere radius=${caster_radius}
- link left_motor: mass 0.0095 -> None; geometry collision box size=${motor_depth} ${motor_width} ${motor_height}; visual box size=${motor_depth} ${motor_width} ${motor_height}
- link left_wheel: mass 0.019 -> None; geometry collision cylinder length=${wheel_width} radius=${wheel_radius}; visual cylinder length=${wheel_width} radius=${wheel_radius}
- link right_motor: mass 0.0095 -> None; geometry collision box size=${motor_depth} ${motor_width} ${motor_height}; visual box size=${motor_depth} ${motor_width} ${motor_height}
- link right_wheel: mass 0.019 -> None; geometry collision cylinder length=${wheel_width} radius=${wheel_radius}; visual cylinder length=${wheel_width} radius=${wheel_radius}
Joints:
- removed joint chassis2caster
- removed joint chassis2left_motor
- removed joint chassis2right_motor
- removed joint left_motor2left_wheel
- removed joint right_motor2right_wheel
- added joint base_link-base_footprint: type fixed, parent base_link, child base_footprint, origin xyz=0.0 0.0 ${-wheel_radius+motor_zoff} rpy=0 0 0
- added joint base_link-base_inertial: type fixed, parent base_link, child base_inertial, origin xyz=0 0 0 rpy=0 0 0
- added joint base_link-caster: type fixed, parent base_link, child caster, origin xyz=${caster_xoff} 0 ${caster_zoff} rpy=0 0 0
- added joint base_link-left_motor: type fixed, parent base_link, child left_motor, origin xyz=0 ${motor_yoff} ${motor_zoff} rpy=0 0 0
- added joint base_link-right_motor: type fixed, parent base_link, child right_motor, origin xyz=0 ${-motor_yoff} ${motor_zoff} rpy=0 0 0
- added joint left_motor-left_wheel: type continuous, parent left_motor, child left_wheel, origin xyz=0 ${motor_width / 2 + motor_shaft_length - wheel_inner_width / 2} 0 rpy=${-pi/2} 0 0, axis 0 0 1
- added joint right_motor-right_wheel: type continuous, parent right_motor, child right_wheel, origin xyz=0 ${-(motor_width / 2 + motor_shaft_length - wheel_inner_width / 2)} 0 rpy=${-pi/2} 0 0, axis 0 0 1

Commit message: add lidar link

File: roundr_description/urdf/roundr.urdf (robot description, URDF)
Before this commit: robot roundr, 8 links, 7 joints
Links:
- removed link caster
- added link front_caster; collision sphere radius=${caster_radius}; visual sphere radius=${caster_radius}
- added link lidar_house; collision cylinder length=0.024 radius=0.035; visual cylinder length=0.024 radius=0.035
- added link lidar_motor; collision cylinder length=0.016 radius=0.016; visual cylinder length=0.016 radius=0.016
- added link rear_caster; collision sphere radius=${caster_radius}; visual sphere radius=${caster_radius}
Joints:
- removed joint base_link-caster
- added joint base_link-front_caster: type fixed, parent base_link, child front_caster, origin xyz=${caster_xoff} 0 ${caster_zoff} rpy=0 0 0
- added joint base_link-lidar_house: type fixed, parent base_link, child lidar_house, origin xyz=0 0 0.092 rpy=0 0 0
- added joint base_link-lidar_motor: type fixed, parent base_link, child lidar_motor, origin xyz=0.045 0 0.072 rpy=0 0 0
- added joint base_link-rear_caster: type fixed, parent base_link, child rear_caster, origin xyz=${-caster_xoff} 0 ${caster_zoff} rpy=0 0 0
